File: Ground_Station_L432_SR105U_FLASH_20261008/Ground_Station_L432_SR105U_FLASH_20261008.kicad_pcb (KiCad board)
At the start: 2 copper layers, 90.2 x 95.9 mm, 159 parts, among them J10 SC1464-ND, J11 SC1464-ND, J12 SQ, J13 Conn_01x12, J15 Conn_01x12, J7 SQ, J8 Conn_01x15, J9 Conn_01x15, SW1 SW_Push, SW2 MODE, SW3 SW_Push, SW4 SW_Coded, U1 SR105U, U3 MCP604, U4 W25Q128JVS

Commit message: Update PCB design. Replace Send button with larger one.
Parts:
- removed SW3: SW_Push, Button_Switch_THT:SW_PUSH_1P1T_6x3.5mm_H4.3_APEM_MJTP1243
- added SW5: SEND, GroundStation:SW_PUSH-12mm, F.Cu at (143.9, 104.6)
- moved TP2 24.0 mm to (80.8, 113.8), turned to 180 degrees
- moved TP1 21.5 mm to (84.1, 113.8), turned to 180 degrees
- moved JP2 19.4 mm to (76.5, 109.7), turned to 90 degrees
- moved SW1 19.3 mm to (67.1, 106.7), turned to 0 degrees
- moved C1 19.2 mm to (80.8, 110.3), turned to -90 degrees
- moved R4 17.0 mm to (83.3, 110.3), turned to 90 degrees
- moved RV1 16.8 mm to (70.3, 116.6), turned to 0 degrees
- moved R11 8.37 mm to (76.4, 116.7), turned to 180 degrees
- moved TP8 7.66 mm to (117.9, 105.5)
- moved TP9 4.75 mm to (117.9, 112.0)
- moved C4 4.28 mm to (132.4, 117.7)
- moved R20 4.28 mm to (132.4, 114.0)
- moved R8 3.84 mm to (128.6, 124.0)
- moved SW4 3.33 mm to (125.5, 114.0)
- moved RN1 3.33 mm to (131.8, 107.2)
- renumbered TX to TP8, RX to TP9
Connections:
- J13 pad 1: (no net) -> /3V3
- J13 pad 10: (no net) -> /3V3
- J13 pad 11: (no net) -> /3V3
- J13 pad 12: (no net) -> /3V3
- J13 pad 2: (no net) -> /3V3
- J13 pad 3: (no net) -> /3V3
- J13 pad 4: (no net) -> /3V3
- J13 pad 5: (no net) -> /3V3
- J13 pad 6: (no net) -> /3V3
- J13 pad 7: (no net) -> /3V3
- J13 pad 8: (no net) -> /3V3
- J13 pad 9: (no net) -> /3V3
Routing:
- net /MIC_IN: track 57.5 -> 76.1 mm
- net Net-(U1-MIC-IN): track 29.0 -> 47.5 mm, vias 1 -> 2
- net /AUDIO_OUT: track 38.0 -> 54.8 mm
- net /SEND: track 47.6 -> 60.1 mm
- net /NRST: track 30.5 -> 36.0 mm
- net /3V3: track 22.7 -> 28.1 mm, vias 4 -> 3
- net /SEL_2: track 59.4 -> 54.2 mm
- net /SEL_1: track 56.9 -> 53.4 mm
- net /SEL_0: track 46.0 -> 42.5 mm
- net Net-(R11-Pad2): track 2.62 -> 5.18 mm
- net /FILTER_OUT: track 11.6 -> 12.8 mm, vias 0 -> 2
- net /UART1_TX: track 93.4 -> 92.4 mm
- net /UART1_RX: track 91.6 -> 90.6 mm
Other:
- board text added: "TSAI@NTUT 20261010"
- board text added: "UART_RX"
- board text added: "UART_TX"
- board text removed: "TSAI@NTUT 20261008"
